Commit message: first commit

File: ros2_ws/src/rse_shl1_description/urdf/shl1_robot_isaac.urdf.xacro (robot description, xacro)
@@ -465,8 +465,14 @@
     </collision>
   </link>
+   <link name="zed2_camera_link"/>
+  <joint name="zed2_camera_mount_joint" type="fixed">
+    <parent link="armario"/>
+    <child link="zed2_camera_link"/>
+    <origin rpy="0 0 0" xyz="0.1 0 0.6925"/>
+  </joint>
   <joint name="zed2_camera_center_joint" type="fixed">
-    <parent link="armario"/>
+    <parent link="zed2_camera_link"/>
     <child link="zed2_camera_center"/>
-    <origin rpy="0.0 0.0 0.0" xyz="0.1 0.0 0.7075"/>
+    <origin rpy="0 0.05 0" xyz="0 0 0.015"/>
   </joint>
   <link name="zed2_left_camera_frame"/>
@@ -474,5 +480,5 @@
     <parent link="zed2_camera_center"/>
     <child link="zed2_left_camera_frame"/>
-    <origin rpy="0 0 0" xyz="0 0.06 0"/>
+    <origin rpy="0 0 0" xyz="-0.01 0.06 0"/>
   </joint>
   <link name="zed2_left_camera_optical_frame"/>
@@ -486,5 +492,5 @@
     <parent link="zed2_camera_center"/>
     <child link="zed2_right_camera_frame"/>
-    <origin rpy="0 0 0" xyz="0 -0.06 0"/>
+    <origin rpy="0 0 0" xyz="-0.01 -0.06 0"/>
   </joint>
   <link name="zed2_right_camera_optical_frame"/>
@@ -493,4 +499,10 @@
     <parent link="zed2_right_camera_frame"/>
     <child link="zed2_right_camera_optical_frame"/>
+  </joint>
+   <link name="zed2_imu_link"/>
+  <joint name="zed2_imu_joint" type="fixed">
+    <parent link="zed2_camera_center"/>
+    <child link="zed2_imu_link"/>
+    <origin xyz="-0.012 0.037 0.000" rpy="-0.000 -0.006 -0.002"/>
   </joint>
   <xacro:front_bumper parent="base_link"/>
